File: Project2.kicad_sch (KiCad schematic)
At the start: 0 parts

Commit message: input progress
Other:
- added sheet Input (input.kicad_sch)
Changed lines of the file:
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@@
 	(paper "A4")
 	(sheet
-		(at 108.585 53.34)
+		(at 76.835 53.975)
+		(size 29.845 23.495)
+		(fields_autoplaced yes)
+		(stroke
+			(width 0.1524)
+			(type solid)
+		)
+		(fill
+			(color 0 0 0 0.0000)
+		)
+		(property "Sheetname" "Input"
+			(at 76.835 53.2634 0)
+			(effects
+				(font
+					(size 1.27 1.27)
+				)
+				(justify left bottom)
+			)
+		)
+		(property "Sheetfile" "input.kicad_sch"
+			(at 76.835 78.0546 0)
+			(effects
+				(font
+					(size 1.27 1.27)
+				)
+				(justify left top)
+			)
+		)
+		(instances
+			(project "Project2"
+				(path "/e8eb11e1-6cec-414d-9150-5cfb3d1c103e"
+					(page "3")
+				)
+			)
+		)
+	)
+	(sheet
+		(at 108.585 53.975)
 		(size 29.845 23.495)
 		(fields_autoplaced yes)
@@
 		)
 		(property "Sheetname" "Microcontroller"
-			(at 108.585 52.6284 0)
+			(at 108.585 53.2634 0)
 			(effects
 				(font
@@
 		)
 		(property "Sheetfile" "mcu.kicad_sch"
-			(at 108.585 77.4196 0)
+			(at 108.585 78.0546 0)
 			(effects
 				(font

Commit message: input schematic update
Other:
- sheet Input ports: added JTAG_TCK, JTAG_TDI, JTAG_TDO, JTAG_TMS, UART_RXD, UART_TXD, UART_TXDEN, UART_~{CTS}, UART_~{DCD}, UART_~{DSR}, UART_~{DTR}, UART_~{RI}, UART_~{RTS}; removed none
Changed lines of the file:
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@@
+			)
+		)
+		(pin "JTAG_TCK" output
+			(at 106.68 57.15 0)
+			(effects
+				(font
+					(size 1.27 1.27)
+				)
+				(justify right)
+			)
+		)
+		(pin "JTAG_TDO" output
+			(at 106.68 59.69 0)
+			(effects
+				(font
+					(size 1.27 1.27)
+				)
+				(justify right)
+			)
+		)
+		(pin "JTAG_TDI" output
+			(at 106.68 62.23 0)
+			(effects
+				(font
+					(size 1.27 1.27)
+				)
+				(justify right)
+			)
+		)
+		(pin "JTAG_TMS" output
+			(at 106.68 64.77 0)
+			(effects
+				(font
+					(size 1.27 1.27)
+				)
+				(justify right)
+			)
+		)
+		(pin "UART_RXD" output
+			(at 106.68 67.31 0)
+			(effects
+				(font
+					(size 1.27 1.27)
+				)
+				(justify right)
+			)
+		)
+		(pin "UART_~{CTS}" output
+			(at 106.68 71.12 0)
+			(effects
+				(font
+					(size 1.27 1.27)
+				)
+				(justify right)
+			)
+		)
+		(pin "UART_~{RTS}" output
+			(at 106.68 73.66 0)
+			(effects
+				(font
+					(size 1.27 1.27)
+				)
+				(justify right)
+			)
+		)
+		(pin "UART_~{DTR}" output
+			(at 76.835 72.39 180)
+			(effects
+				(font
+					(size 1.27 1.27)
+				)
+				(justify left)
+			)
+		)
+		(pin "UART_TXD" output
+			(at 76.835 69.85 180)
+			(effects
+				(font
+					(size 1.27 1.27)
+				)
+				(justify left)
+			)
+		)
+		(pin "UART_~{DCD}" output
+			(at 76.835 67.31 180)
+			(effects
+				(font
+					(size 1.27 1.27)
+				)
+				(justify left)
+			)
+		)
+		(pin "UART_~{RI}" output
+			(at 76.835 64.77 180)
+			(effects
+				(font
+					(size 1.27 1.27)
+				)
+				(justify left)
+			)
+		)
+		(pin "UART_TXDEN" output
+			(at 76.835 62.23 180)
+			(effects
+				(font
+					(size 1.27 1.27)
+				)
+				(justify left)
+			)
+		)
+		(pin "UART_~{DSR}" output
+			(at 76.835 59.69 180)
+			(effects
+				(font
+					(size 1.27 1.27)
+				)
+				(justify left)
 			)
 		)
