File: Project2.kicad_pcb (KiCad board)
At the start: 2 copper layers, 100 x 100 mm, 2 parts, among them U1 ESP32-S3-WROOM-1-N16R2

Commit message: input progress
Parts:
- added J1: USB4105-GF-A, AA_Connectors:GCT_USB4105-GF-A, F.Cu at (112.7, 83.5)
- added U2: FT2232HL, AA_USB_Interface:QFP50P1200X1200X160-64N, F.Cu at (114.8, 69.5)
Other:
- copper layers 2 -> 4
