File: Project2.kicad_pcb (KiCad board)
At the start: 4 copper layers, 100 x 100 mm, 11 parts, among them J1 USB4105-GF-A, U1 ESP32-S3-WROOM-1-N16R2, U2 FT2232HL

Commit message: Add files via upload
Parts:
- removed D1: DSS14U, AA_Diodes:SOD-123FL
- removed D2: ESDA6V1BC6, Package_TO_SOT_SMD:SOT-23-6
- removed J1: USB4105-GF-A, AA_Connectors:GCT_USB4105-GF-A
- removed U1: ESP32-S3-WROOM-1-N16R2, AA_MCUs:ESP32S3WROOM1N16R2
- added C10: 22uF, Capacitor_SMD:C_0805_2012Metric_Pad1.18x1.45mm_HandSolder, F.Cu at (121.0, 112.0)
- added C11: 22uF, Capacitor_SMD:C_0805_2012Metric_Pad1.18x1.45mm_HandSolder, F.Cu at (118.0, 112.0)
- added C12: 22uF, Capacitor_SMD:C_0805_2012Metric_Pad1.18x1.45mm_HandSolder, F.Cu at (114.5, 112.0)
- added C18: 1nF, Capacitor_SMD:C_0805_2012Metric_Pad1.18x1.45mm_HandSolder, F.Cu at (126.0, 93.0)
- added C19: 10uF, Capacitor_SMD:C_0805_2012Metric_Pad1.18x1.45mm_HandSolder, F.Cu at (96.0, 96.5)
- added C21: 10uF, Capacitor_SMD:C_0805_2012Metric_Pad1.18x1.45mm_HandSolder, F.Cu at (99.0, 96.5)
- added C23: 100nF, Capacitor_SMD:C_0805_2012Metric_Pad1.18x1.45mm_HandSolder, F.Cu at (104.5, 92.5)
- added C25: 22uF, Capacitor_SMD:C_0805_2012Metric_Pad1.18x1.45mm_HandSolder, F.Cu at (113.5, 92.5)
- added C27: 22uF, Capacitor_SMD:C_0805_2012Metric_Pad1.18x1.45mm_HandSolder, F.Cu at (113.5, 94.5)
- added C6: 100nF, Capacitor_SMD:C_0805_2012Metric_Pad1.18x1.45mm_HandSolder, F.Cu at (138.5, 96.5)
- added C7: 10uF, Capacitor_SMD:C_0805_2012Metric_Pad1.18x1.45mm_HandSolder, F.Cu at (94.0, 112.0)
- added C8: 10uF, Capacitor_SMD:C_0805_2012Metric_Pad1.18x1.45mm_HandSolder, F.Cu at (97.0, 112.0)
- added C9: 100nF, Capacitor_SMD:C_0805_2012Metric_Pad1.18x1.45mm_HandSolder, F.Cu at (102.5, 108.5)
- added IC1: KP256XTMA2, Weather Station:KP256XTMA2, F.Cu at (147.1, 97.6)
- added L1: 3.3uH, Inductor_SMD:L_1008_2520Metric_Pad1.43x2.20mm_HandSolder, F.Cu at (107.5, 107.0)
- added L3: 3.3uH, Inductor_SMD:L_1008_2520Metric_Pad1.43x2.20mm_HandSolder, F.Cu at (109.0, 91.0)
- added R11: 33k, Resistor_SMD:R_0805_2012Metric_Pad1.20x1.40mm_HandSolder, F.Cu at (107.5, 112.0)
- added R13: 10k, Resistor_SMD:R_0805_2012Metric_Pad1.20x1.40mm_HandSolder, F.Cu at (111.0, 113.0)
- added R5: 10k, Resistor_SMD:R_0805_2012Metric_Pad1.20x1.40mm_HandSolder, F.Cu at (115.0, 98.0)
- added U3: TPS562201DDCR, Weather Station:DDC0006A_M, F.Cu at (102.0, 112.1)
- added U4: TPS562201DDCR, Weather Station:DDC0006A_M, F.Cu at (104.0, 96.6)
- C16: value 8p -> 100nF; footprint Capacitor_SMD:C_0805_2012Metric -> Capacitor_SMD:C_0805_2012Metric_Pad1.18x1.45mm_HandSolder
- C17: value 8p -> 1nF; footprint Capacitor_SMD:C_0805_2012Metric -> Capacitor_SMD:C_0805_2012Metric_Pad1.18x1.45mm_HandSolder
- R1: value 5.1k -> R_Photo; footprint Resistor_SMD:R_0805_2012Metric -> Weather Station:photores
- R2: value 5.1k -> R; footprint Resistor_SMD:R_0805_2012Metric -> Resistor_SMD:R_0805_2012Metric_Pad1.20x1.40mm_HandSolder
- R3: value 4.7k -> 51k; footprint Resistor_SMD:R_0805_2012Metric -> Resistor_SMD:R_0805_2012Metric_Pad1.20x1.40mm_HandSolder
- R4: value 10k -> 5.1k; footprint Resistor_SMD:R_0805_2012Metric -> Resistor_SMD:R_0805_2012Metric_Pad1.20x1.40mm_HandSolder
- U2: value FT2232HL -> SHT31-ARP-B; footprint AA_USB_Interface:QFP50P1200X1200X160-64N -> Weather Station:SHT31-ARP-B_SEN
- moved R2 62.1 mm to (136.5, 102.5)
- moved R1 60.1 mm to (130.5, 102.5), turned to 180 degrees
- moved C16 51.6 mm to (135.0, 96.5), turned to -90 degrees
- moved C17 43.6 mm to (126.0, 97.0), turned to -90 degrees
- moved R4 38.2 mm to (112.0, 98.0), turned to -90 degrees
- moved R3 37.5 mm to (109.0, 96.0), turned to -90 degrees
- moved U2 29.8 mm to (130.8, 94.7)
Connections:
- C16 pad 1: /Microcontroller/XTAL_32K_P -> 3.3V
- C17 pad 1: /Microcontroller/XTAL_32K_N -> Temperature
- R1 pad 1: GND -> light
- R1 pad 2: /Input/USB_CC2 -> 3.3V
- R2 pad 1: GND -> light
- R2 pad 2: /Input/USB_CC1 -> GND
- R3 pad 1: /Input/~{PWRSAV} -> Net-(SW1-C)
- R3 pad 2: VBUS -> Net-(R3-Pad2)
- R4 pad 1: GND -> Net-(R3-Pad2)
- R4 pad 2: /Input/~{PWRSAV} -> Net-(U4-VFB)
- U2 pad 1: GND -> Humidity
- U2 pad 2: unconnected-(U2-OSCI-Pad2) -> GND
- U2 pad 3: unconnected-(U2-OSCO-Pad3) -> GND
- U2 pad 4: unconnected-(U2-VPHY-Pad4) -> Temperature
- U2 pad 5: GND -> 3.3V
- U2 pad 7: unconnected-(U2-D--Pad7) -> GND
- U2 pad 8: unconnected-(U2-D+-Pad8) -> GND
- U2 pad 9: unconnected-(U2-VPLL-Pad9) -> GND
Routing:
- net 3.3V: track 0.00 -> 49.7 mm
- net Net-(U4-SW): track 0.00 -> 12.7 mm
- net GND: track 0.00 -> 12.7 mm, vias 0 -> 2
- net Net-(U3-SW): track 0.00 -> 12.6 mm
- net Net-(U4-VFB): track 0.00 -> 10.2 mm
- net 12V: track 0.00 -> 9.86 mm
- net 5V: track 0.00 -> 9.84 mm
- net Net-(C10-Pad2): track 0.00 -> 9.02 mm
- net Net-(SW1-C): track 0.00 -> 8.30 mm
- net Net-(U3-VFB): track 0.00 -> 6.55 mm
- net Net-(C25-Pad2): track 0.00 -> 4.69 mm
- net Temperature: track 0.00 -> 3.70 mm
- net Humidity: track 0.00 -> 3.53 mm
- net light: track 0.00 -> 3.30 mm
- net Net-(U4-VBST): track 0.00 -> 3.14 mm
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- added copper zone on F.Cu, net GND
Other:
- outline, holes or cut-outs redrawn
