File: _autosave-Project2.kicad_pcb (KiCad board)
At the start: 4 copper layers, 100 x 100 mm, 11 parts, among them J1 USB4105-GF-A, U1 ESP32-S3-WROOM-1-N16R2, U2 FT2232HL

Commit message: input schematic update
Routing:
- net GND: track 0.00 -> 13.3 mm
Changed lines of the file:
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@@
 		(tags "SOT TO_SOT_SMD")
 		(property "Reference" "D2"
-			(at 0 -2.4 360)
+			(at 0 -2.4 0)
 			(layer "F.SilkS")
 			(effects
@@
 		)
 		(property "Value" "ESDA6V1BC6"
-			(at 0 2.4 360)
+			(at 0 2.4 0)
 			(layer "F.Fab")
 			(effects
@@
 		)
 		(fp_text user "${REFERENCE}"
-			(at 0 0 360)
+			(at 0 0 0)
 			(layer "F.Fab")
 			(effects
@@
 		(layer "Edge.Cuts")
 	)
+	(segment
+		(start 84.755 83.8)
+		(end 88.605 79.95)
+		(width 0.2)
+		(layer "F.Cu")
+		(net 1)
+	)
+	(segment
+		(start 88.605 79.95)
+		(end 96.5 79.95)
+		(width 0.2)
+		(layer "F.Cu")
+		(net 1)
+	)
 )
