File: mcu.kicad_sch (KiCad schematic)
At the start: 20 parts, among them U1 ESP32-S2FN4R2, Y1 ECX-1637B2

Commit message: mcu update
Parts:
- removed C1, C7: 1u, symbol Device:C
- removed C10, C11: 8p, symbol Device:C
- removed C2, C5, C6, C8, C9: 0.1u, symbol Device:C
- removed C4: 100p, symbol Device:C
- removed L2: 24n, symbol Device:L
- removed U1: ESP32-S2FN4R2, symbol AA_MCUs:ESP32-S2FN4R2
- removed Y1: ECX-1637B2, ECX1637B2, symbol AA_Crystals:ECX-1637B2
- added C16, C17: 8p, symbol Device:C
- added U1: ESP32-S3-WROOM-1-N16R2, symbol AA_MCUs:ESP32-S3-WROOM-1-N16R2
- added Y2: CFS-206 (32kHz RTC), CFS-206, symbol AA_Crystals:CFS-206
Connections:
- net GND renamed EPAD
- net EPAD: now also C16.2, C17.2, U1.1 (GND), U1.40 (GND), U1.41 (EPAD)
- new net XTAL_32K_N: C17.1, U1.9 (IO16), Y2.2 (XOUT)
- new net XTAL_32K_P: C16.1, U1.8 (IO15), Y2.1 (XIN)
Other:
- note added: "Crystal"
- note removed: "Crystal Oscillator"

Commit message: input progress
Parts:
- removed D1: ESD9B5.0ST5G, Diode_SMD:D_SOD-923, symbol Diode:ESD9B5.0ST5G
- U1: footprint (none) -> AA_MCUs:ESP32S3WROOM1N16R2
Changed lines of the file:
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@@
-	(wire
-		(pts
-			(xy 266.7 40.64) (xy 266.7 41.91)
-		)
-		(stroke
-			(width 0)
-			(type default)
-		)
-	)
 	(wire
 		(pts
@@
 		(pts
 			(xy 66.04 31.75) (xy 66.04 36.83)
-		)
-		(stroke
-			(width 0)
-			(type default)
-		)
-	)
-	(wire
-		(pts
-			(xy 266.7 31.75) (xy 266.7 33.02)
 		)
 		(stroke
@@
 			)
 		)
-		(property "Footprint" ""
+		(property "Footprint" "AA_MCUs:ESP32S3WROOM1N16R2"
 			(at 170.942 22.606 0)
 			(effects
@@
 					(unit 1)
 				)
-			)
-		)
-	)
-	(symbol
-		(lib_id "power:+3.3V")
-		(at 266.7 31.75 0)
-		(unit 1)
-		(exclude_from_sim no)
-		(in_bom yes)
-		(on_board yes)
-		(dnp no)
-		(fields_autoplaced yes)
-		(property "Reference" "#PWR06"
-			(at 266.7 35.56 0)
-			(effects
-				(font
-					(size 1.27 1.27)
-				)
-				(hide yes)
-			)
-		)
-		(property "Value" "+3.3V"
-			(at 266.7 26.67 0)
-			(effects
-				(font
-					(size 1.27 1.27)
-				)
-			)
-		)
-		(property "Footprint" ""
-			(at 266.7 31.75 0)
-			(effects
-				(font
-					(size 1.27 1.27)
-				)
-				(hide yes)
-			)
-		)
-		(property "Datasheet" ""
-			(at 266.7 31.75 0)
-			(effects
-				(font
-					(size 1.27 1.27)
-				)
-				(hide yes)
-			)
-		)
-		(property "Description" "Power symbol creates a global label with name \"+3.3V\""
-			(at 266.7 31.75 0)
-			(effects
-				(font
-					(size 1.27 1.27)
-				)
-				(hide yes)
-			)
-		)
-		(pin "1"
-		)
-		(instances
-			(project "Project2"
-				(path "/e8eb11e1-6cec-414d-9150-5cfb3d1c103e/db1ed3d3-f9ac-49e3-915b-45158cabfd8f"
-					(reference "#PWR06")
-					(unit 1)
-				)
-			)
-		)
-	)
-	(symbol
-		(lib_id "power:GND")
-		(at 266.7 41.91 0)
-		(unit 1)
-		(exclude_from_sim no)
-		(in_bom yes)
-		(on_board yes)
-		(dnp no)
-		(fields_autoplaced yes)
-		(property "Reference" "#PWR07"
-			(at 266.7 48.26 0)
-			(effects
-				(font
-					(size 1.27 1.27)
-				)
-				(hide yes)
-			)
-		)
-		(property "Value" "GND"
-			(at 266.7 46.99 0)
-			(effects
-				(font
-					(size 1.27 1.27)
-				)
-			)
-		)
-		(property "Footprint" ""
-			(at 266.7 41.91 0)
-			(effects
-				(font
-					(size 1.27 1.27)
-				)
-				(hide yes)
-			)
-		)
-		(property "Datasheet" ""
-			(at 266.7 41.91 0)
-			(effects
-				(font
-					(size 1.27 1.27)
-				)
-				(hide yes)
-			)
-		)
-		(property "Description" "Power symbol creates a global label with name \"GND\" , ground"
-			(at 266.7 41.91 0)
-			(effects
-				(font
-					(size 1.27 1.27)
-				)
-				(hide yes)
-			)
-		)
-		(pin "1"
-		)
-		(instances
-			(project ""
-				(path "/e8eb11e1-6cec-414d-9150-5cfb3d1c103e/db1ed3d3-f9ac-49e3-915b-45158cabfd8f"
-					(reference "#PWR07")
-					(unit 1)
-				)
-			)
-		)
-	)
-	(symbol
-		(lib_id "Diode:ESD9B5.0ST5G")
-		(at 266.7 36.83 90)
-		(unit 1)
-		(exclude_from_sim no)
-		(in_bom yes)
-		(on_board yes)
-		(dnp no)
-		(fields_autoplaced yes)
-		(property "Reference" "D1"
-			(at 269.24 35.5599 90)
-			(effects
-				(font
-					(size 1.27 1.27)
-				)
-				(justify right)
-			)
-		)
-		(property "Value" "ESD9B5.0ST5G"
-			(at 269.24 38.0999 90)
-			(effects
-				(font
-					(size 1.27 1.27)
-				)
-				(justify right)
-			)
-		)
-		(property "Footprint" "Diode_SMD:D_SOD-923"
-			(at 266.7 36.83 0)
-			(effects
-				(font
-					(size 1.27 1.27)
-				)
-				(hide yes)
-			)
-		)
-		(property "Datasheet" "https://www.onsemi.com/pub/Collateral/ESD9B-D.PDF"
-			(at 266.7 36.83 0)
-			(effects
-				(font
-					(size 1.27 1.27)
-				)
-				(hide yes)
-			)
-		)
-		(property "Description" "ESD protection diode, 5.0Vrwm, SOD-923"
-			(at 266.7 36.83 0)
-			(effects
-				(font
-					(size 1.27 1.27)
-				)
-				(hide yes)
-			)
-		)
-		(pin "2"
-		)
-		(pin "1"
-		)
-		(instances
-			(project ""
-				(path "/e8eb11e1-6cec-414d-9150-5cfb3d1c103e/db1ed3d3-f9ac-49e3-915b-45158cabfd8f"
-					(reference "D1")
-					(unit 1)
-				)

Commit message: input schematic update
Parts:
- removed C12: 10u, symbol Device:C
- removed C13: 1u, symbol Device:C
- removed C14, C15: 0.1u, symbol Device:C
- removed C3: C, symbol Device:C
- removed L1: 2n, symbol Device:L
- C16, C17: footprint (none) -> Capacitor_SMD:C_0805_2012Metric
Other:
- note removed: "Decoupling Capacitors"
- note removed: "ESD Protection"
- moved on the sheet: C16, C17
